Commit message: Update: Modifico la posicion de las colisiones para que coincidan con las ruedas

File: my_robot_description/urdf/mobile_base.xacro (robot description, xacro)
@@ -91,5 +91,5 @@
     </visual>
     <collision>
-      <origin xyz="0 0 0" rpy="1.5708 0 0"/>
+      <origin xyz="0 -0.013 0" rpy="1.5708 0 0"/>
       <geometry>
         <cylinder radius="${wheel_radius}" length="0.025"/>
@@ -97,5 +97,5 @@
     </collision>
     <xacro:cylinder_inertia m="0.1403" r="${wheel_radius}" h="0.025"
-                            o_xyz="0 0 0" o_rpy="1.5708 0 0"/>
+                            o_xyz="0 -0.013 0" o_rpy="1.5708 0 0"/>
   </link>
   <link name="Rueda_derecha_link">
@@ -108,5 +108,5 @@
     </visual>
     <collision>
-      <origin xyz="0 0 0" rpy="1.5708 0 0"/>
+      <origin xyz="0 0.013 0" rpy="1.5708 0 0"/>
       <geometry>
         <cylinder radius="${wheel_radius}" length="0.025"/>
@@ -114,5 +114,5 @@
     </collision>
     <xacro:cylinder_inertia m="0.1403" r="${wheel_radius}" h="0.025"
-                            o_xyz="0 0 0" o_rpy="1.5708 0 0"/>
+                            o_xyz="0 0.013 0" o_rpy="1.5708 0 0"/>
   </link>
   <link name="Base_castor_link">
@@ -183,5 +183,5 @@
     <parent link="base_link"/>
     <child link="Lidar_link"/>
-    <origin xyz="0 0 0.05" rpy="0 0 0"/>
+    <origin xyz="0 0 0" rpy="0 0 0"/>
     <axis xyz="0 1 0"/>
   </joint>

Commit message: Update:  Nivelo robot para que no este inclinado y agrego imu

File: my_robot_description/urdf/mobile_base.xacro (robot description, xacro)
@@ -31,19 +31,21 @@
   <xacro:property name="castor_base_scale" value="${global_scale} ${global_scale} ${global_scale}"/>
   <xacro:property name="castor_base_xyz" value="0.072581 0 -0.0025"/>
-  <xacro:property name="castor_base_rpy" value="0 0 0"/>
+  <xacro:property name="castor_base_rpy" value="3.14 3.14 3.14"/>
   <xacro:property name="castor_base_axis" value="0 0 1"/>
-  <xacro:property name="castor_base_visual_rpy"  value="3.14159 0 3.14159"/>
+  <xacro:property name="castor_base_visual_xyz" value="0 0 0"/>
+  <xacro:property name="castor_base_visual_rpy" value="0 3.14 0"/>
   <!-- Rueda castor -->
   <xacro:property name="castor_wheel_mesh" value="Rueda_castor_link.STL"/>
   <xacro:property name="castor_wheel_scale" value="${global_scale} ${global_scale} ${global_scale}"/>
   <xacro:property name="castor_wheel_xyz" value="-0.015014 -0.00012272 -0.02296"/>
-  <xacro:property name="castor_wheel_rpy" value="0 0 0"/>
+  <xacro:property name="castor_wheel_rpy" value="3.14 3.14 -3.14"/>
   <xacro:property name="castor_wheel_axis" value="0 1 0"/>
-  <xacro:property name="castor_wheel_visual_rpy" value="1.5708 0 0"/>
+  <xacro:property name="castor_wheel_visual_xyz" value="0 0 0"/>
+  <xacro:property name="castor_wheel_visual_rpy" value="1.5708 0.042481 0"/>
   <!-- Parámetros geométricos de referencia para usar en control/TF -->
   <!-- No se usan explicitamente, pero sirven para dejar documentadas las dimensiones principales -->
   <xacro:property name="wheel_separation" value="0.1605"/>
-  <xacro:property name="wheel_radius" value="0.033"/>
-  <xacro:property name="robot_length" value="0.185"/>
+  <xacro:property name="wheel_radius" value="0.0345"/>
+  <xacro:property name="robot_length" value="0.2"/>
   <xacro:property name="robot_width" value="0.145"/>
   <xacro:property name="robot_height" value="0.050"/>
@@ -131,7 +133,7 @@
     </collision>
     <inertial>
-      <mass value="0.01"/>
+      <mass value="0.1"/>
       <origin xyz="0 0 0" rpy="0 0 0"/>
-      <inertia ixx="1e-6" ixy="0" ixz="0" iyy="1e-6" iyz="0" izz="1e-6"/>
+      <inertia ixx="1e-4" ixy="0" ixz="0" iyy="1e-4" iyz="0" izz="1e-4"/>
     </inertial>
   </link>
@@ -145,13 +147,32 @@
     </visual>
     <collision>
-      <origin xyz="0 0 0" rpy="0 0 0"/>
-      <geometry>
-        <sphere radius="0.01"/>
+      <origin xyz="0 0 0" rpy="1.5708 0 0"/>
+      <geometry>
+        <cylinder radius="0.015" length="0.015"/>
+      </geometry>
+    </collision>
+    <xacro:cylinder_inertia m="0.01" r="0.015" h="0.01"
+                            o_xyz="0 0 0" o_rpy="0 0 0"/>
+  </link>
+  <link name="caja_castor_link">
+    <visual>
+      <origin xyz="0 0 -0.0062" rpy="${castor_base_visual_rpy}" />
+      <geometry>
+        <box size="0.03 0.03 0.015" />
+      </geometry>
+      <material name="Cyan">
+        <color rgba="0 1.0 1.0 1.0"/>
+      </material>
+    </visual>
+    <collision>
+      <origin xyz="0 0 -0.0062" rpy="0 0 0"/>
+      <geometry>
+        <box size="0.03 0.03 0.015" />
       </geometry>
     </collision>
     <inertial>
-      <mass value="0.005"/>
-      <origin xyz="0 0 0" rpy="0 0 0"/>
-      <inertia ixx="1e-6" ixy="0" ixz="0" iyy="1e-6" iyz="0" izz="1e-6"/>
+      <mass value="0.1"/>
+      <origin xyz="0 0 0." rpy="0 0 0"/>
+      <inertia ixx="1e-4" ixy="0" ixz="0" iyy="1e-4" iyz="0" izz="1e-4"/>
     </inertial>
   </link>
@@ -159,5 +180,5 @@
   <link name="Lidar_link">
     <visual>
-      <origin xyz="0 0 0.01" rpy="0 0 0"/>
+      <origin xyz="0 0 0.0095" rpy="0 0 0"/>
       <geometry>
         <cylinder radius="0.025" length="0.02"/>
@@ -168,5 +189,5 @@
     </visual>
     <collision>
-      <origin xyz="0 0 0.01" rpy="0 0 0"/>
+      <origin xyz="0 0 0.005" rpy="0 0 0"/>
       <geometry>
         <cylinder radius="0.025" length="0.02"/>
@@ -174,16 +195,17 @@
     </collision>
     <inertial>
-      <mass value="0.01"/>
-      <origin xyz="0 0 0.01" rpy="0 0 0"/>
-      <inertia ixx="1e-6" ixy="0" ixz="0" iyy="1e-6" iyz="0" izz="1e-6"/>
+      <mass value="0.1"/>
+      <origin xyz="0 0 0.005" rpy="0 0 0"/>
+      <inertia ixx="1e-4" ixy="0" ixz="0" iyy="1e-4" iyz="0" izz="1e-4"/>
     </inertial>
   </link>
-  <!-- Joint que fija el LIDAR al chasis -->
-  <joint name="Lidar_joint" type="fixed">
-    <parent link="base_link"/>
-    <child link="Lidar_link"/>
-    <origin xyz="0 0 0" rpy="0 0 0"/>
-    <axis xyz="0 1 0"/>
-  </joint>
+  <link name="imu_link">
+    <visual>
+      <geometry>
+        <box size="0.02 0.02 0.01"/>
+      </geometry>
+      <material name="blue"/>
+    </visual>
+  </link>
  <!-- Instancia Link rueda derecha-->
   <joint name="Rueda_derecha_joint" type="continuous">
@@ -193,8 +215,20 @@
     <axis xyz="${right_wheel_axis}"/>
   </joint>
- <!-- Instancia Link caja castor-->
+  <joint name="Rueda_izquierda_joint" type="continuous">
+    <origin xyz="${left_wheel_xyz}" rpy="${left_wheel_rpy}"/>
+    <parent link="base_link"/>
+    <child link="Rueda_izquierda_link"/>
+    <axis xyz="${left_wheel_axis}"/>
+  </joint>
+  <joint name="caja_castor_joint" type="fixed">
+    <origin xyz="${castor_base_xyz}" rpy="${castor_base_rpy}"/>
+    <parent link="base_link"/>
+    <child link="caja_castor_link"/>
+    <axis xyz="${castor_base_axis}"/>
+  </joint>
+ <!-- Instancia Link base castor-->
   <joint name="Base_castor_joint" type="continuous">
-    <origin xyz="${castor_base_xyz}" rpy="${castor_base_rpy}"/>
-    <parent link="base_link"/>
+    <origin xyz="0 0 -0.008" rpy="${castor_base_rpy}"/>
+    <parent link="caja_castor_link"/>
     <child link="Base_castor_link"/>
     <axis xyz="${castor_base_axis}"/>
@@ -207,15 +241,21 @@
     <axis xyz="${castor_wheel_axis}"/>
   </joint>
-  <!-- Joints -->
+    <!-- Joint que fija el LIDAR al chasis -->
+  <joint name="Lidar_joint" type="fixed">
+    <parent link="base_link"/>
+    <child link="Lidar_link"/>
+    <origin xyz="0 0 0" rpy="0 0 0"/>
+    <axis xyz="0 1 0"/>
+  </joint>
+  <joint name="imu_joint" type="fixed">
+    <parent link="Lidar_link"/>
+    <child link="imu_link"/>
+    <origin xyz="0 0 0.02" rpy="0 0 0"/>
+  </joint>
+    <!-- Joints -->
   <joint name="base_joint" type="fixed">
-  <parent link="base_footprint"/>
-  <child link="base_link"/>
-  <origin xyz="0 0 0.04675" rpy="0 0 0"/>
-  </joint>
-  <joint name="Rueda_izquierda_joint" type="continuous">
-    <origin xyz="${left_wheel_xyz}" rpy="${left_wheel_rpy}"/>
-    <parent link="base_link"/>
-    <child link="Rueda_izquierda_link"/>
-    <axis xyz="${left_wheel_axis}"/>
+    <parent link="base_footprint"/>
+    <child link="base_link"/>
+    <origin xyz="0 0 0.04675" rpy="0 0 0"/>
   </joint>
 </robot>

File: my_robot_description/urdf/my_robot_gazebo.xacro (robot description, xacro)
@@ -36,5 +36,6 @@
   <gazebo reference="Lidar_link">
     <sensor name="gpu_lidar" type="gpu_lidar">
-      <pose relative_to="Lidar_link">0 0 0.01 0 0 0</pose>
+      <!-- <pose relative_to="Lidar_link">0 0 0.01 0 0 0</pose> -->
+      <pose>0 0 0 0 0 0</pose>
       <always_on>true</always_on>
       <visualize>true</visualize>
@@ -68,3 +69,11 @@
     <preserveFixedJoint>true</preserveFixedJoint>
   </gazebo>
+  <gazebo reference="imu_link">
+    <sensor name="imu_sensor" type="imu">
+      <always_on>1</always_on>
+      <update_rate>100</update_rate>
+      <visualize>true</visualize>
+      <topic>imu</topic>
+    </sensor>
+  </gazebo>
 </robot>

Commit message: Update: Corrijo integracion de imu y actualizo las especificaciones del lidar a las del rplidar a1

File: my_robot_description/urdf/mobile_base.xacro (robot description, xacro)
@@ -245,5 +245,5 @@
     <parent link="base_link"/>
     <child link="Lidar_link"/>
-    <origin xyz="0 0 0" rpy="0 0 0"/>
+    <origin xyz="0 0 0" rpy="0 -0.00478 0"/>
     <axis xyz="0 1 0"/>
   </joint>

File: my_robot_description/urdf/my_robot_gazebo.xacro (robot description, xacro)
@@ -34,7 +34,6 @@
   </gazebo>
   <!-- Sensor LIDAR asociado al link -->
-  <gazebo reference="Lidar_link">
+  <!-- <gazebo reference="Lidar_link">
     <sensor name="gpu_lidar" type="gpu_lidar">
-      <!-- <pose relative_to="Lidar_link">0 0 0.01 0 0 0</pose> -->
       <pose>0 0 0 0 0 0</pose>
       <always_on>true</always_on>
@@ -64,8 +63,49 @@
       </lidar>
     </sensor>
+  </gazebo> -->
+  <!-- Nuevo sensor LIDAR (RPLIDAR A1) asociado al Link_lidar-->
+  <gazebo reference="Lidar_link">
+    <sensor name="gpu_lidar" type="gpu_lidar">
+      <always_on>true</always_on>
+      <visualize>true</visualize>
+      <update_rate>5.5</update_rate>
+      <topic>scan</topic>
+      <gz_frame_id>Lidar_link</gz_frame_id>
+      <lidar>
+        <scan>
+          <horizontal>
+            <samples>1450</samples>
+            <resolution>1.0</resolution>
+            <min_angle>-3.14159</min_angle>
+            <max_angle>3.14159</max_angle>
+          </horizontal>
+          <vertical>
+            <samples>1</samples>
+            <resolution>1.0</resolution>
+            <min_angle>0.0</min_angle>
+            <max_angle>0.0</max_angle>
+          </vertical>
+        </scan>
+        <range>
+          <min>0.15</min>
+          <max>12.0</max>
+          <resolution>0.001</resolution>
+        </range>
+        <noise>
+          <type>gaussian</type>
+          <mean>0.0</mean>
+          <stddev>0.03</stddev>
+        </noise>
+      </lidar>
+    </sensor>
   </gazebo>
   <!-- Evita que Gazebo fusione el joint fijo del LIDAR -->
   <gazebo reference="Lidar_joint">
     <preserveFixedJoint>true</preserveFixedJoint>
+  </gazebo>
+  <gazebo>
+    <plugin filename="gz-sim-imu-system"
+            name="gz::sim::systems::Imu">
+    </plugin>
   </gazebo>
   <gazebo reference="imu_link">

Commit message: Update: Reduzco los valores de inercia de los links relacionados a la rueda castor

File: my_robot_description/urdf/mobile_base.xacro (robot description, xacro)
@@ -133,7 +133,8 @@
     </collision>
     <inertial>
-      <mass value="0.1"/>
+      <mass value="0.005"/>
       <origin xyz="0 0 0" rpy="0 0 0"/>
-      <inertia ixx="1e-4" ixy="0" ixz="0" iyy="1e-4" iyz="0" izz="1e-4"/>
+      <inertia ixx="2e-7" ixy="0" ixz="0" iyy="2e-7" iyz="0" izz="2e-7"/>
+      <!-- <inertia ixx="1e-4" ixy="0" ixz="0" iyy="1e-4" iyz="0" izz="1e-4"/> -->
     </inertial>
   </link>
@@ -152,6 +153,7 @@
       </geometry>
     </collision>
-    <xacro:cylinder_inertia m="0.01" r="0.015" h="0.01"
-                            o_xyz="0 0 0" o_rpy="0 0 0"/>
+    <xacro:cylinder_inertia m="0.005" r="0.015" h="0.015" o_xyz="0 0 0" o_rpy="0 0 0"/>
+    <!-- <xacro:cylinder_inertia m="0.01" r="0.015" h="0.01"
+                            o_xyz="0 0 0" o_rpy="0 0 0"/> -->
   </link>
   <link name="caja_castor_link">
@@ -172,7 +174,8 @@
     </collision>
     <inertial>
-      <mass value="0.1"/>
+      <mass value="0.005"/>
       <origin xyz="0 0 0." rpy="0 0 0"/>
-      <inertia ixx="1e-4" ixy="0" ixz="0" iyy="1e-4" iyz="0" izz="1e-4"/>
+      <inertia ixx="4.68e-7" ixy="0" ixz="0" iyy="4.68e-7" iyz="0" izz="7.5e-7"/>
+      <!-- <inertia ixx="1e-4" ixy="0" ixz="0" iyy="1e-4" iyz="0" izz="1e-4"/> -->
     </inertial>
   </link>
@@ -195,7 +198,8 @@
     </collision>
     <inertial>
-      <mass value="0.1"/>
+      <mass value="0.015"/>
       <origin xyz="0 0 0.005" rpy="0 0 0"/>
-      <inertia ixx="1e-4" ixy="0" ixz="0" iyy="1e-4" iyz="0" izz="1e-4"/>
+      <inertia ixx="2.84e-6" ixy="0" ixz="0" iyy="2.84e-6" iyz="0" izz="4.69e-6"/>
+      <!-- <inertia ixx="1e-4" ixy="0" ixz="0" iyy="1e-4" iyz="0" izz="1e-4"/> -->
     </inertial>
   </link>
