Commit message: EKF (ruedas + IMU) y arbitro Tremaux: el robot resuelve el laberinto
Localizacion:
- imu_link y plugin IMU (100 Hz) en el Xacro; /imu agregado al bridge.
- ekf_filter_node (robot_localization) con ekf.yaml: fusiona velocidades de
  rueda con el yaw del giroscopo. Publica /odometry/filtered y la TF
  odom -> base_footprint.
- publish_odom_tf: false en el diff-drive (evita doble publicacion de TF).
- Corregida la altura de la rueda castor (cabeceo que desviaba el rayo
  frontal del LIDAR hacia el piso).

Navegacion:
- El nodo pasa a suscribirse a /odometry/filtered.
- GIRO_U transiciona a POST_GIRO con reset de contador (antes salia
  directo a AVANZAR, arrastrando el error angular del giro de 180).
- Grilla de celdas visitadas (0.45 m, la constante de red del laberinto)
  y metricas de tiempo y distancia recorrida.
- Arbitro Tremaux: entre las direcciones libres segun el LIDAR, elige la
  celda vecina menos visitada; la mano derecha queda como desempate.
- Frontera virtual (celda_valida): excluye las celdas fuera del laberinto
  de las opciones del arbitro.
- Detector de meta por coordenadas: el robot se detiene sobre el disco y
  reporta tiempo, distancia y celdas exploradas.

Simulacion:
- El launch usa maze_2.world y spawnea el robot en el disco rojo (entrada).
- package.xml de bringup: se declaran las dependencias de ejecucion.

File: my_robot_description/urdf/mobile_base.xacro (robot description, xacro)
@@ -30,5 +30,5 @@
   <xacro:property name="castor_base_mesh" value="Base_castor_link.STL"/>
   <xacro:property name="castor_base_scale" value="${global_scale} ${global_scale} ${global_scale}"/>
-  <xacro:property name="castor_base_xyz" value="0.072581 0 -0.0025"/>
+  <xacro:property name="castor_base_xyz" value="0.072581 0 -0.009"/>
   <xacro:property name="castor_base_rpy" value="0 0 0"/>
   <xacro:property name="castor_base_axis" value="0 0 1"/>
@@ -186,4 +186,18 @@
     <axis xyz="0 1 0"/>
   </joint>
+  <!-- Link de la IMU, sensor puntual, sin geometria visible -->
+  <link name="imu_link">
+    <inertial>
+      <mass value="0.001"/>
+      <origin xyz="0 0 0" rpy="0 0 0"/>
+      <inertia ixx="1e-7" ixy="0" ixz="0" iyy="1e-7" iyz="0" izz="1e-7"/>
+    </inertial>
+  </link>
+  <!-- Joint que fija la IMU al chasis, en el centro de rotacion -->
+  <joint name="imu_joint" type="fixed">
+    <parent link="base_link"/>
+    <child link="imu_link"/>
+    <origin xyz="0 0 0.02" rpy="0 0 0"/>
+  </joint>
  <!-- Instancia Link rueda derecha-->
   <joint name="Rueda_derecha_joint" type="continuous">

File: my_robot_description/urdf/my_robot_gazebo.xacro (robot description, xacro)
@@ -12,4 +12,5 @@
       <frame_id>odom</frame_id>
       <child_frame_id>base_footprint</child_frame_id>
+      <publish_odom_tf>false</publish_odom_tf>
     </plugin>
   </gazebo>
@@ -40,5 +41,5 @@
       <visualize>true</visualize>
       <topic>scan</topic>
-      <update_rate>2</update_rate>
+      <update_rate>10</update_rate>
       <gz_frame_id>Lidar_link</gz_frame_id>
       <lidar>
@@ -68,3 +69,18 @@
     <preserveFixedJoint>true</preserveFixedJoint>
   </gazebo>
+  <!-- Plugin del sistema IMU de Gazebo -->
+  <gazebo>
+    <plugin filename="gz-sim-imu-system"
+            name="gz::sim::systems::Imu">
+    </plugin>
+  </gazebo>
+  <!-- Sensor IMU asociado al imu_link -->
+  <gazebo reference="imu_link">
+    <sensor name="imu_sensor" type="imu">
+      <always_on>true</always_on>
+      <update_rate>100</update_rate>
+      <topic>imu</topic>
+      <gz_frame_id>imu_link</gz_frame_id>
+    </sensor>
+  </gazebo>
 </robot>
