Commit message: Update: Ajusto mi modelo para que pueda funcionar con el wall_following

File: my_robot_description/urdf/mobile_base_abi.xacro (robot description, xacro)
@@ -133,8 +133,9 @@
     </collision>
     <inertial>
-      <mass value="0.005"/>
-      <origin xyz="0 0 0" rpy="0 0 0"/>
-      <inertia ixx="2e-7" ixy="0" ixz="0" iyy="2e-7" iyz="0" izz="2e-7"/>
+      <mass value="0.01"/>
+      <origin xyz="0 0 0" rpy="0 0 0"/>
+      <!-- <inertia ixx="2e-7" ixy="0" ixz="0" iyy="2e-7" iyz="0" izz="2e-7"/> -->
       <!-- <inertia ixx="1e-4" ixy="0" ixz="0" iyy="1e-4" iyz="0" izz="1e-4"/> -->
+      <inertia ixx="1e-6" ixy="0" ixz="0" iyy="1e-6" iyz="0" izz="1e-6"/>
     </inertial>
   </link>
@@ -175,7 +176,6 @@
     <inertial>
       <mass value="0.005"/>
-      <origin xyz="0 0 0." rpy="0 0 0"/>
-      <inertia ixx="4.68e-7" ixy="0" ixz="0" iyy="4.68e-7" iyz="0" izz="7.5e-7"/>
-      <!-- <inertia ixx="1e-4" ixy="0" ixz="0" iyy="1e-4" iyz="0" izz="1e-4"/> -->
+      <origin xyz="0 0 0" rpy="0 0 0"/>
+      <inertia ixx="1e-6" ixy="0" ixz="0" iyy="1e-6" iyz="0" izz="1e-6"/>
     </inertial>
   </link>
@@ -198,19 +198,18 @@
     </collision>
     <inertial>
-      <mass value="0.015"/>
+      <mass value="0.01"/>
+      <origin xyz="0 0 0.01" rpy="0 0 0"/>
+      <inertia ixx="1e-6" ixy="0" ixz="0" iyy="1e-6" iyz="0" izz="1e-6"/>
+    </inertial>
+  </link>
+  <link name="Imu_link">
+    <visual>
+      <geometry>
+        <box size="0.02 0.02 0.01"/>
+      </geometry>
+      <material name="blue"/>
+    </visual>
+    <collision>
       <origin xyz="0 0 0.005" rpy="0 0 0"/>
-      <inertia ixx="2.84e-6" ixy="0" ixz="0" iyy="2.84e-6" iyz="0" izz="4.69e-6"/>
-      <!-- <inertia ixx="1e-4" ixy="0" ixz="0" iyy="1e-4" iyz="0" izz="1e-4"/> -->
-    </inertial>
-  </link>
-  <link name="imu_link">
-    <visual>
-      <geometry>
-        <box size="0.02 0.02 0.01"/>
-      </geometry>
-      <material name="blue"/>
-    </visual>
-    <collision>
-      <origin xyz="0 0 0.005" rpy="0 0 0"/>
       <geometry>
         <cylinder radius="0.025" length="0.02"/>
@@ -218,8 +217,7 @@
     </collision>
     <inertial>
-      <mass value="0.015"/>
-      <origin xyz="0 0 0.005" rpy="0 0 0"/>
-      <inertia ixx="2.84e-6" ixy="0" ixz="0" iyy="2.84e-6" iyz="0" izz="4.69e-6"/>
-      <!-- <inertia ixx="1e-4" ixy="0" ixz="0" iyy="1e-4" iyz="0" izz="1e-4"/> -->
+      <mass value="0.005"/>
+      <origin xyz="0 0 0" rpy="0 0 0"/>
+      <inertia ixx="1e-6" ixy="0" ixz="0" iyy="1e-6" iyz="0" izz="1e-6"/>
     </inertial>
   </link>
@@ -264,7 +262,7 @@
     <axis xyz="0 1 0"/>
   </joint>
-  <joint name="imu_joint" type="fixed">
-    <parent link="base_link"/>
-    <child link="imu_link"/>
+  <joint name="Imu_joint" type="fixed">
+    <parent link="base_link"/>
+    <child link="Imu_link"/>
     <origin xyz="0 0 -0.005" rpy="0 0 0"/>
   </joint>

File: my_robot_description/urdf/my_robot_abi_gazebo.xacro (robot description, xacro)
@@ -10,6 +10,4 @@
       <wheel_separation>${wheel_separation}</wheel_separation>
       <wheel_radius>${wheel_radius}</wheel_radius>
-      <odom_topic>odom</odom_topic>
-      <odom_publish_frequency>30</odom_publish_frequency>
       <frame_id>odom</frame_id>
       <child_frame_id>base_footprint</child_frame_id>
@@ -20,5 +18,5 @@
       filename="gz-sim-odometry-publisher-system"
       name="gz::sim::systems::OdometryPublisher">
-      <odom_frame>odom</odom_frame>
+      <odom_frame>world</odom_frame>
       <robot_base_frame>base_footprint</robot_base_frame>
       <odom_topic>/real_odom</odom_topic>
@@ -46,6 +44,7 @@
   </gazebo>
   <!-- Nuevo sensor LIDAR (RPLIDAR A1) asociado al Link_lidar-->
-  <gazebo reference="Lidar_link">
+  <!-- <gazebo reference="Lidar_link">
     <sensor name="gpu_lidar" type="gpu_lidar">
+      <pose relative_to="Lidar_link">0 0 0.01 0 0 0</pose>
       <always_on>true</always_on>
       <visualize>true</visualize>
@@ -80,4 +79,34 @@
       </lidar>
     </sensor>
+  </gazebo> -->
+  <gazebo reference="Lidar_link">
+    <sensor name="gpu_lidar" type="gpu_lidar">
+      <pose relative_to="Lidar_link">0 0 0.01 0 0 0</pose>
+      <always_on>true</always_on>
+      <visualize>true</visualize>
+      <topic>scan</topic>
+      <update_rate>2</update_rate>
+      <gz_frame_id>Lidar_link</gz_frame_id>
+      <lidar>
+        <scan>
+          <horizontal>
+            <samples>180</samples>
+            <resolution>1.0</resolution>
+            <min_angle>0.0</min_angle>
+            <max_angle>6.28</max_angle>
+          </horizontal>
+        </scan>
+        <range>
+          <min>0.12</min>
+          <max>12.0</max>
+          <resolution>0.02</resolution>
+        </range>
+        <noise>
+          <type>gaussian</type>
+          <mean>0.0</mean>
+          <stddev>0.01</stddev>
+        </noise>
+      </lidar>
+    </sensor>
   </gazebo>
   <!-- Evita que Gazebo fusione el joint fijo del LIDAR -->
@@ -90,7 +119,7 @@
     </plugin>
   </gazebo>
-  <gazebo reference="imu_link">
+  <gazebo reference="Imu_link">
     <sensor name="imu_sensor" type="imu">
-      <gz_frame_id>Lidar_link</gz_frame_id>
+      <gz_frame_id>Imu_link</gz_frame_id>
       <always_on>1</always_on>
       <update_rate>100</update_rate>

Commit message: Fix: Finalmente el topico de /odometry/filtered coincide con la grilla y en rviz el robot  va por encima del camino que pinta el mapa

File: my_robot_description/urdf/mobile_base_abi.xacro (robot description, xacro)
@@ -67,5 +67,5 @@
   <!-- Sin geometria, punto de contacto del robot con el suelo -->
   <link name="base_footprint"/>
-   <link name="base_link">
+  <link name="base_link">
     <visual>
       <origin xyz="${base_visual_xyz}" rpy="${base_visual_rpy}"/>
@@ -82,5 +82,5 @@
     </collision>
     <xacro:box_inertia m="0.12" x="${robot_length}" y="${robot_width}" z="${robot_height}"
-                       o_xyz="0 0 0" o_rpy="0 0 0"/>
+                        o_xyz="0 0 0" o_rpy="0 0 0"/>
   </link>
   <link name="Rueda_izquierda_link">
@@ -149,7 +149,7 @@
     </visual>
     <collision>
-      <origin xyz="0 0 0" rpy="1.5708 0 0"/>
-      <geometry>
-        <cylinder radius="0.015" length="0.015"/>
+      <origin xyz="0 0 0" rpy="0 0 0"/>
+      <geometry>
+        <sphere radius="0.015"/>
       </geometry>
     </collision>

File: my_robot_description/urdf/my_robot_abi_gazebo.xacro (robot description, xacro)
@@ -10,7 +10,8 @@
       <wheel_separation>${wheel_separation}</wheel_separation>
       <wheel_radius>${wheel_radius}</wheel_radius>
+      <odom_topic>/wheel_odom</odom_topic>
+      <tf_topic>/gazebo_internal/tf</tf_topic>
       <frame_id>odom</frame_id>
       <child_frame_id>base_footprint</child_frame_id>
-      <publish_odom_tf>false</publish_odom_tf>
     </plugin>
   </gazebo>
@@ -45,5 +46,5 @@
   </gazebo>
   <!-- Nuevo sensor LIDAR (RPLIDAR A1) asociado al Link_lidar-->
-  <!-- <gazebo reference="Lidar_link">
+  <gazebo reference="Lidar_link">
     <sensor name="gpu_lidar" type="gpu_lidar">
       <pose relative_to="Lidar_link">0 0 0.01 0 0 0</pose>
@@ -80,6 +81,6 @@
       </lidar>
     </sensor>
-  </gazebo> -->
-  <gazebo reference="Lidar_link">
+  </gazebo>
+  <!-- <gazebo reference="Lidar_link">
     <sensor name="gpu_lidar" type="gpu_lidar">
       <pose relative_to="Lidar_link">0 0 0.01 0 0 0</pose>
@@ -110,5 +111,5 @@
       </lidar>
     </sensor>
-  </gazebo>
+  </gazebo> -->
   <!-- Evita que Gazebo fusione el joint fijo del LIDAR -->
   <gazebo reference="Lidar_joint">
